File: frontpanel.brd (EAGLE design)
At the start: 21 x 87 mm, 45 parts, among them J1 HD_AUDIO, J2 CTRL, J3 RST_SW, J4 PWR_LED, J5 HDD_LED, J6 SW_LED, J7 MIC, J8 HP, Q1 NMOSL, Q2 NMOSL, Q3 PMOS, Q4 PMOS, Q5 PMOS, SW1 RST, U1 CPC1006N, U2 CPC1006N, U3 CPC1006N, U4 CPC1006N

Commit message: Parts Ordered
Parts:
- J7, J8: device BW-Connectors:ACJS-NV35-5 -> BW-Connectors:ACJS-MV35-5
- R10, R7: value 4.7kΩ -> 2kΩ
- U1, U2, U3, U4: value CPC1006N -> CPC1017N; device BW-Active:CPC1006N -> BW-Active:CPC10*N
Changed lines of the file:
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@@
 <layer number="48" name="Document" color="7" fill="1" visible="yes" active="yes"/>
 <layer number="49" name="Reference" color="7" fill="1" visible="yes" active="yes"/>
+<layer number="50" name="dxf" color="7" fill="1" visible="no" active="no"/>
 <layer number="51" name="tDocu" color="7" fill="1" visible="yes" active="yes"/>
 <layer number="52" name="bDocu" color="7" fill="1" visible="yes" active="yes"/>
@@
 <layer number="98" name="Guide" color="6" fill="1" visible="no" active="no"/>
 <layer number="99" name="SpiceOrder" color="5" fill="1" visible="no" active="no"/>
+<layer number="250" name="Descript" color="3" fill="1" visible="no" active="no"/>
+<layer number="251" name="SMDround" color="12" fill="11" visible="no" active="no"/>
 </layers>
 <board>
-<fusionsync huburn="a.cGVyc29uYWw6dWUyYmY1N2E4" projecturn="a.cGVyc29uYWw6dWUyYmY1N2E4IzIwMjIwMTIwNDg3Nzg3NTgx" f3durn="urn:adsk.wipprod:dm.lineage:TSz83DG2Q-msOJfVkx_v7g" pcbguid="" lastpulledtime="" lastsyncedchangeguid="" latestrevisionid="0ba3b859-e271-4129-8f01-a1532b939d05" lastsyncedrevisionid="0ba3b859-e271-4129-8f01-a1532b939d05" lastboardhashguid="18cc49b1-a552-ead0-d879-1fbbab7b1ec7" lastpushedtime="2022-02-08T18:33:26Z" linktopcb3d="true"/>
+<fusionsync huburn="a.cGVyc29uYWw6dWUyYmY1N2E4" projecturn="a.cGVyc29uYWw6dWUyYmY1N2E4IzIwMjIwMTIwNDg3Nzg3NTgx" f3durn="urn:adsk.wipprod:dm.lineage:TSz83DG2Q-msOJfVkx_v7g" pcbguid="" lastpulledtime="" lastsyncedchangeguid="" latestrevisionid="93165bb4-4907-44d5-bfa0-c8a3bc8672d5" lastsyncedrevisionid="93165bb4-4907-44d5-bfa0-c8a3bc8672d5" lastboardhashguid="c17c3de9-f9ca-41f0-d9cb-a886b428a5c7" lastpushedtime="2022-02-19T19:56:35Z" linktopcb3d="true"/>
 <plain>
 <wire x1="0" y1="0" x2="21" y2="0" width="0" layer="20"/>
@@
 <attribute name="VALUE" x="14.185" y="0.715" size="1.27" layer="27" font="vector" ratio="12" rot="R90"/>
 </element>
-<element name="J7" library="BW-Connectors" library_urn="urn:adsk.eagle:library:33858393" package="ACJS-NV35-5" package3d_urn="urn:adsk.eagle:package:33935525/5" value="MIC" x="10.5" y="56" smashed="yes">
+<element name="J7" library="BW-Connectors" library_urn="urn:adsk.eagle:library:33858393" package="ACJS-MV35-5" package3d_urn="urn:adsk.eagle:package:33935524/3" value="MIC" x="10.5" y="56" smashed="yes">
 <attribute name="NAME" x="17.96" y="49.97" size="1.016" layer="25" font="vector" ratio="15"/>
 <attribute name="VALUE" x="16.56" y="48.23" size="1.016" layer="27" font="vector" ratio="15"/>
 </element>
-<element name="J8" library="BW-Connectors" library_urn="urn:adsk.eagle:library:33858393" package="ACJS-NV35-5" package3d_urn="urn:adsk.eagle:package:33935525/5" value="HP" x="10.5" y="39.6" smashed="yes">
+<element name="J8" library="BW-Connectors" library_urn="urn:adsk.eagle:library:33858393" package="ACJS-MV35-5" package3d_urn="urn:adsk.eagle:package:33935524/3" value="HP" x="10.5" y="39.6" smashed="yes">
 <attribute name="NAME" x="18.06" y="33.47" size="1.016" layer="25" font="vector" ratio="15"/>
 <attribute name="VALUE" x="16.56" y="31.83" size="1.016" layer="27" font="vector" ratio="15"/>
@@
 <attribute name="VALUE" x="16.135" y="73.195" size="1.016" layer="28" font="vector" ratio="15" rot="MR0"/>
 </element>
-<element name="R10" library="resistor" library_urn="urn:adsk.eagle:library:348" package="R0603" package3d_urn="urn:adsk.eagle:package:23555/3" value="4.7kΩ" x="4.1" y="34.7" smashed="yes" rot="MR270">
+<element name="R10" library="resistor" library_urn="urn:adsk.eagle:library:348" package="R0603" package3d_urn="urn:adsk.eagle:package:23555/3" value="2kΩ" x="4.1" y="34.7" smashed="yes" rot="MR270">
 <attribute name="NAME" x="2.235" y="33.465" size="1.016" layer="26" font="vector" ratio="15" rot="MR90"/>
-<attribute name="VALUE" x="0.995" y="32.865" size="1.016" layer="28" font="vector" ratio="15" rot="MR90"/>
+<attribute name="VALUE" x="0.895" y="33.465" size="1.016" layer="28" font="vector" ratio="15" rot="MR90"/>
 </element>
 <element name="R11" library="resistor" library_urn="urn:adsk.eagle:library:348" package="R0603" package3d_urn="urn:adsk.eagle:package:23555/3" value="470kΩ" x="7.6" y="30.7" smashed="yes" rot="MR0">
@@
 <attribute name="VALUE" x="15.035" y="55.695" size="1.016" layer="28" font="vector" ratio="15" rot="MR0"/>
 </element>
-<element name="R7" library="resistor" library_urn="urn:adsk.eagle:library:348" package="R0603" package3d_urn="urn:adsk.eagle:package:23555/3" value="4.7kΩ" x="4.1" y="51.3" smashed="yes" rot="MR270">
+<element name="R7" library="resistor" library_urn="urn:adsk.eagle:library:348" package="R0603" package3d_urn="urn:adsk.eagle:package:23555/3" value="2kΩ" x="4.1" y="51.3" smashed="yes" rot="MR270">
 <attribute name="NAME" x="2.235" y="50.565" size="1.016" layer="26" font="vector" ratio="15" rot="MR90"/>
-<attribute name="VALUE" x="0.995" y="49.465" size="1.016" layer="28" font="vector" ratio="15" rot="MR90"/>
+<attribute name="VALUE" x="0.995" y="49.965" size="1.016" layer="28" font="vector" ratio="15" rot="MR90"/>
 </element>
 <element name="R8" library="resistor" library_urn="urn:adsk.eagle:library:348" package="R0603" package3d_urn="urn:adsk.eagle:package:23555/3" value="470kΩ" x="7.4" y="47.2" smashed="yes" rot="MR0">
@@
 <attribute name="VALUE" x="15.7" y="72.8" size="1.016" layer="27" font="vector" ratio="15"/>
 </element>
-<element name="U1" library="BW-Active" library_urn="urn:adsk.eagle:library:33783073" package="CPC1006N" package3d_urn="urn:adsk.eagle:package:33936582/2" value="CPC1006N" x="8.9" y="55.9" smashed="yes" rot="MR90">
+<element name="U1" library="BW-Active" library_urn="urn:adsk.eagle:library:33783073" package="CPC10*N" package3d_urn="urn:adsk.eagle:package:33936582/3" value="CPC1017N" x="8.9" y="55.9" smashed="yes" rot="MR90">
 <attribute name="NAME" x="12.84" y="52.64" size="1.016" layer="26" font="vector" ratio="15" rot="MR0"/>
 <attribute name="VALUE" x="18.167" y="53.944" size="1.016" layer="28" font="vector" ratio="15" rot="MR0"/>
 </element>
-<element name="U2" library="BW-Active" library_urn="urn:adsk.eagle:library:33783073" package="CPC1006N" package3d_urn="urn:adsk.eagle:package:33936582/2" value="CPC1006N" x="9" y="39" smashed="yes" rot="MR90">
+<element name="U2" library="BW-Active" library_urn="urn:adsk.eagle:library:33783073" package="CPC10*N" package3d_urn="urn:adsk.eagle:package:33936582/3" value="CPC1017N" x="9" y="39" smashed="yes" rot="MR90">
 <attribute name="NAME" x="12.74" y="35.54" size="1.016" layer="26" font="vector" ratio="15" rot="MR0"/>
 <attribute name="VALUE" x="18.267" y="37.044" size="1.016" layer="28" font="vector" ratio="15" rot="MR0"/>
 </element>
-<element name="U3" library="BW-Active" library_urn="urn:adsk.eagle:library:33783073" package="CPC1006N" package3d_urn="urn:adsk.eagle:package:33936582/2" value="CPC1006N" x="16" y="19.1" smashed="yes" rot="MR90">
+<element name="U3" library="BW-Active" library_urn="urn:adsk.eagle:library:33783073" package="CPC10*N" package3d_urn="urn:adsk.eagle:package:33936582/3" value="CPC1017N" x="16" y="19.1" smashed="yes" rot="MR90">
 <attribute name="NAME" x="15.44" y="15.16" size="1.016" layer="26" font="vector" ratio="15" rot="MR90"/>
 <attribute name="VALUE" x="18.444" y="15.833" size="1.016" layer="28" font="vector" ratio="15" rot="MR90"/>
 </element>
-<element name="U4" library="BW-Active" library_urn="urn:adsk.eagle:library:33783073" package="CPC1006N" package3d_urn="urn:adsk.eagle:package:33936582/2" value="CPC1006N" x="4.6" y="16.9" smashed="yes" rot="MR270">
+<element name="U4" library="BW-Active" library_urn="urn:adsk.eagle:library:33783073" package="CPC10*N" package3d_urn="urn:adsk.eagle:package:33936582/3" value="CPC1017N" x="4.6" y="16.9" smashed="yes" rot="MR270">
 <attribute name="NAME" x="4.04" y="13.06" size="1.016" layer="26" font="vector" ratio="15" rot="MR90"/>
 <attribute name="VALUE" x="1.144" y="13.533" size="1.016" layer="28" font="vector" ratio="15" rot="MR90"/>

Commit message: Miscellaneous progress
Parts:
- removed Q3, Q4, Q5: PMOS, BW-Active:SOT23
- added D1, D2, D3, D4: BAT60A, BW-Active:SOD323
- added U5: 7414PW, BW-Active:TSSOP14
- J6: device pinhead:1X04/90 -> pinhead:1X04
- LED1: device BW-Active:L1MC-RGB0035000MP0 -> BW-Active:PLCC-6
- R1: value 1kΩ? -> 1kΩ
- R10, R7: value 2kΩ -> 510Ω
- R11, R8: value 470kΩ -> 100kΩ
- R18, R19: value 1kΩ -> 510Ω
- R6, R9: value 1kΩ? -> 0Ω
- U1, U2, U3, U4: value CPC1017N -> G3VM-61VY3; device BW-Active:CPC10*N -> BW-Active:SOP-4
- moved R6 6.72 mm to (7.40, 62.7)
- moved J6 3.72 mm to (7.10, 10.9), flipped to the bottom, turned to 0 degrees
- moved U3 2.00 mm to (16.0, 21.1), turned to 0 degrees
- moved U1 1.75 mm to (9.30, 57.6), turned to 315 degrees
- moved U2 1.30 mm to (9.00, 40.3), turned to 0 degrees
- moved U4 0.10 mm to (4.70, 16.9), turned to 180 degrees
Connections:
- removed net LED_B: Q5.3, R14.2, R17.1
- removed net LED_G: Q4.3, R13.2, R16.1
- removed net LED_R: Q3.3, R12.2, R15.1
- new net HDD_LED_B_RAW: R14.2, U5.12
- new net HDD_LED_G_RAW: R13.2, U5.10
- new net HDD_LED_R_RAW: R12.2, U5.8
- new net SW_LED_B_RAW: R17.1, U5.2
- new net SW_LED_G_RAW: R16.1, U5.4
- new net SW_LED_R_RAW: R15.1, U5.6
- net !PWM_B: now also U5.1, U5.13; no longer Q5.1
- net !PWM_G: now also U5.11, U5.3; no longer Q4.1
- net !PWM_R: now also U5.5, U5.9; no longer Q3.1
- net 5V: now also U5.14; no longer Q3.2, Q4.2, Q5.2
- net AUD_GND: no longer Q1.2, Q2.2
- net GND: now also Q1.2, Q2.2, U5.7
- net HDD_LED_DRIVE: now also D1.1
- net HDD_LED_IN-: now also D1.2
- net HP_SENSEDR_A: now also D4.1
- net HP_SENSEDR_K: now also D4.2
- net MIC_SENSEDR_A: now also D3.1
- net MIC_SENSEDR_K: now also D3.2
- net PWR_LED_IN-: now also D2.2
- net SW_LED_DRIVE: now also D2.1
Routing:
- net GND: track 0.00 -> 36.2 mm, vias 8 -> 18
- net LED_B: track 23.8 -> 0.00 mm
- net LED_G: track 22.9 -> 0.00 mm
- net LED_R: track 15.1 -> 0.00 mm
- net SW_LED_B_RAW: track 0.00 -> 10.7 mm
- net 5V: track 58.1 -> 47.6 mm
- net SW_LED_G_RAW: track 0.00 -> 8.69 mm
- net !PWM_B: track 9.57 -> 16.5 mm
- net HDD_LED_B_RAW: track 0.00 -> 6.67 mm
- net SW_LED_R_RAW: track 0.00 -> 6.57 mm
- net HDD_LED_G_RAW: track 0.00 -> 5.78 mm
- net SW_LED_DRIVE: track 3.91 -> 9.59 mm
- net MIC_SENSEDR_A: track 6.79 -> 12.3 mm
- net !PWM_G: track 11.3 -> 16.5 mm
- net HDD_LED_R_RAW: track 0.00 -> 3.54 mm
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- added copper zone on layer 1, net LOGO
- removed copper zone on layer 16, net LOGO
Other:
- board text added: "JLCJLCJLCJLC"
