File: frontpanel.sch (EAGLE design)
At the start: 45 parts, among them J1 HD_AUDIO, J2 CTRL, J3 RST_SW, J4 PWR_LED, J5 HDD_LED, J6 SW_LED, J7 MIC, J8 HP, Q1 NMOSL, Q2 NMOSL, Q3 PMOS, Q4 PMOS, Q5 PMOS, SW1 RST, U1 CPC1006N, U2 CPC1006N, U3 CPC1006N, U4 CPC1006N

Commit message: Parts Ordered
Parts:
- J7, J8: device BW-Connectors:ACJS-NV35-5 -> BW-Connectors:ACJS-MV35-5-
- R10, R7: value 4.7kΩ -> 2kΩ
- U1, U2, U3, U4: value CPC1006N -> CPC1017N; device BW-Active:CPC1006N -> BW-Active:CPC1017N
Changed lines of the file:
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@@
 <layer number="48" name="Document" color="7" fill="1" visible="no" active="no"/>
 <layer number="49" name="Reference" color="7" fill="1" visible="no" active="no"/>
+<layer number="50" name="dxf" color="7" fill="1" visible="no" active="no"/>
 <layer number="51" name="tDocu" color="7" fill="1" visible="no" active="no"/>
 <layer number="52" name="bDocu" color="7" fill="1" visible="no" active="no"/>
@@
 <layer number="98" name="Guide" color="6" fill="1" visible="yes" active="yes"/>
 <layer number="99" name="SpiceOrder" color="5" fill="1" visible="yes" active="yes"/>
+<layer number="250" name="Descript" color="3" fill="1" visible="no" active="no"/>
+<layer number="251" name="SMDround" color="12" fill="11" visible="no" active="no"/>
 </layers>
 <schematic xreflabel="%F%N/%S.%C%R" xrefpart="/%S.%C%R">
@@
 <part name="J5" library="pinhead" library_urn="urn:adsk.eagle:library:325" deviceset="PINHD-1X2" device="" package3d_urn="urn:adsk.eagle:package:22435/2" value="HDD_LED"/>
 <part name="J6" library="pinhead" library_urn="urn:adsk.eagle:library:325" deviceset="PINHD-1X4" device="/90" package3d_urn="urn:adsk.eagle:package:22404/2" value="SW_LED"/>
-<part name="J7" library="BW-Connectors" library_urn="urn:adsk.eagle:library:33858393" deviceset="ACJS-*V35-5" device="" package3d_urn="urn:adsk.eagle:package:33935525/5" technology="N" value="MIC"/>
-<part name="J8" library="BW-Connectors" library_urn="urn:adsk.eagle:library:33858393" deviceset="ACJS-*V35-5" device="" package3d_urn="urn:adsk.eagle:package:33935525/5" technology="N" value="HP"/>
+<part name="J7" library="BW-Connectors" library_urn="urn:adsk.eagle:library:33858393" deviceset="ACJS-*V35-5" device="-" package3d_urn="urn:adsk.eagle:package:33935524/3" technology="M" value="MIC"/>
+<part name="J8" library="BW-Connectors" library_urn="urn:adsk.eagle:library:33858393" deviceset="ACJS-*V35-5" device="-" package3d_urn="urn:adsk.eagle:package:33935524/3" technology="M" value="HP"/>
 <part name="R1" library="resistor" library_urn="urn:adsk.eagle:library:348" deviceset="R-US_" device="R0603" package3d_urn="urn:adsk.eagle:package:23555/3" value="1kΩ?"/>
 <part name="R2" library="resistor" library_urn="urn:adsk.eagle:library:348" deviceset="R-US_" device="R0603" package3d_urn="urn:adsk.eagle:package:23555/3" value="4.7kΩ"/>
@@
 <part name="R4" library="resistor" library_urn="urn:adsk.eagle:library:348" deviceset="R-US_" device="R0603" package3d_urn="urn:adsk.eagle:package:23555/3" value="4.7kΩ"/>
 <part name="R5" library="resistor" library_urn="urn:adsk.eagle:library:348" deviceset="R-US_" device="R0603" package3d_urn="urn:adsk.eagle:package:23555/3" value="4.7kΩ"/>
-<part name="U1" library="BW-Active" library_urn="urn:adsk.eagle:library:33783073" deviceset="CPC1006N" device="" package3d_urn="urn:adsk.eagle:package:33936582/2"/>
-<part name="U2" library="BW-Active" library_urn="urn:adsk.eagle:library:33783073" deviceset="CPC1006N" device="" package3d_urn="urn:adsk.eagle:package:33936582/2"/>
+<part name="U1" library="BW-Active" library_urn="urn:adsk.eagle:library:33783073" deviceset="CPC1017N" device="" package3d_urn="urn:adsk.eagle:package:33936582/3"/>
+<part name="U2" library="BW-Active" library_urn="urn:adsk.eagle:library:33783073" deviceset="CPC1017N" device="" package3d_urn="urn:adsk.eagle:package:33936582/3"/>
 <part name="Q1" library="BW-Active" library_urn="urn:adsk.eagle:library:33783073" deviceset="SOT23-N-MOSFET" device="" package3d_urn="urn:adsk.eagle:package:33783194/2" value="NMOSL"/>
 <part name="Q2" library="BW-Active" library_urn="urn:adsk.eagle:library:33783073" deviceset="SOT23-N-MOSFET" device="" package3d_urn="urn:adsk.eagle:package:33783194/2" value="NMOSL"/>
 <part name="R6" library="resistor" library_urn="urn:adsk.eagle:library:348" deviceset="R-US_" device="R0603" package3d_urn="urn:adsk.eagle:package:23555/3" value="1kΩ?"/>
-<part name="R7" library="resistor" library_urn="urn:adsk.eagle:library:348" deviceset="R-US_" device="R0603" package3d_urn="urn:adsk.eagle:package:23555/3" value="4.7kΩ"/>
+<part name="R7" library="resistor" library_urn="urn:adsk.eagle:library:348" deviceset="R-US_" device="R0603" package3d_urn="urn:adsk.eagle:package:23555/3" value="2kΩ"/>
 <part name="R8" library="resistor" library_urn="urn:adsk.eagle:library:348" deviceset="R-US_" device="R0603" package3d_urn="urn:adsk.eagle:package:23555/3" value="470kΩ"/>
 <part name="R9" library="resistor" library_urn="urn:adsk.eagle:library:348" deviceset="R-US_" device="R0603" package3d_urn="urn:adsk.eagle:package:23555/3" value="1kΩ?"/>
-<part name="R10" library="resistor" library_urn="urn:adsk.eagle:library:348" deviceset="R-US_" device="R0603" package3d_urn="urn:adsk.eagle:package:23555/3" value="4.7kΩ"/>
+<part name="R10" library="resistor" library_urn="urn:adsk.eagle:library:348" deviceset="R-US_" device="R0603" package3d_urn="urn:adsk.eagle:package:23555/3" value="2kΩ"/>
 <part name="R11" library="resistor" library_urn="urn:adsk.eagle:library:348" deviceset="R-US_" device="R0603" package3d_urn="urn:adsk.eagle:package:23555/3" value="470kΩ"/>
 <part name="Q3" library="BW-Active" library_urn="urn:adsk.eagle:library:33783073" deviceset="SOT23-P-MOSFET" device="" package3d_urn="urn:adsk.eagle:package:33783194/2" value="PMOS"/>
@@
 <part name="R16" library="resistor" library_urn="urn:adsk.eagle:library:348" deviceset="R-US_" device="R0603" package3d_urn="urn:adsk.eagle:package:23555/3" value="330Ω"/>
 <part name="R17" library="resistor" library_urn="urn:adsk.eagle:library:348" deviceset="R-US_" device="R0603" package3d_urn="urn:adsk.eagle:package:23555/3" value="330Ω"/>
-<part name="U3" library="BW-Active" library_urn="urn:adsk.eagle:library:33783073" deviceset="CPC1006N" device="" package3d_urn="urn:adsk.eagle:package:33936582/2"/>
-<part name="U4" library="BW-Active" library_urn="urn:adsk.eagle:library:33783073" deviceset="CPC1006N" device="" package3d_urn="urn:adsk.eagle:package:33936582/2"/>
+<part name="U3" library="BW-Active" library_urn="urn:adsk.eagle:library:33783073" deviceset="CPC1017N" device="" package3d_urn="urn:adsk.eagle:package:33936582/3"/>
+<part name="U4" library="BW-Active" library_urn="urn:adsk.eagle:library:33783073" deviceset="CPC1017N" device="" package3d_urn="urn:adsk.eagle:package:33936582/3"/>
 <part name="R18" library="resistor" library_urn="urn:adsk.eagle:library:348" deviceset="R-US_" device="R0603" package3d_urn="urn:adsk.eagle:package:23555/3" value="1kΩ"/>
 <part name="R19" library="resistor" library_urn="urn:adsk.eagle:library:348" deviceset="R-US_" device="R0603" package3d_urn="urn:adsk.eagle:package:23555/3" value="1kΩ"/>

Commit message: Miscellaneous progress
Parts:
- removed Q3, Q4, Q5: PMOS, BW-Active:SOT23-P-MOSFET
- added D1, D2, D3, D4: BAT60A, BW-Active:SOD323-SCHOTTKY
- added U5: 7414PW, BW-Active:7414PW
- J6: device pinhead:PINHD-1X4/90 -> pinhead:PINHD-1X4
- LED1: device BW-Active:L1MC-RGB0035000MP0 -> BW-Active:PLCC-6-RGBLED
- R1: value 1kΩ? -> 1kΩ
- R10, R7: value 2kΩ -> 510Ω
- R11, R8: value 470kΩ -> 100kΩ
- R18, R19: value 1kΩ -> 510Ω
- R6, R9: value 1kΩ? -> 0Ω
- U1, U2, U3, U4: value CPC1017N -> G3VM-61VY3; device BW-Active:CPC1017N -> BW-Active:SOP-4-SSR
Connections:
- removed net LED_B: Q5.D, R14.2, R17.1
- removed net LED_G: Q4.D, R13.2, R16.1
- removed net LED_R: Q3.D, R12.2, R15.1
- new net HDD_LED_B_RAW: R14.2, U5F.O
- new net HDD_LED_G_RAW: R13.2, U5E.O
- new net HDD_LED_R_RAW: R12.2, U5D.O
- new net SW_LED_B_RAW: R17.1, U5A.O
- new net SW_LED_G_RAW: R16.1, U5B.O
- new net SW_LED_R_RAW: R15.1, U5C.O
- net !PWM_B: now also U5A.I, U5F.I; no longer Q5.G
- net !PWM_G: now also U5B.I, U5E.I; no longer Q4.G
- net !PWM_R: now also U5C.I, U5D.I; no longer Q3.G
- net 5V: now also U5P.VCC; no longer Q3.S, Q4.S, Q5.S
- net AUD_GND: no longer Q1.S, Q2.S
- net GND: now also Q1.S, Q2.S, U5P.GND
- net HDD_LED_DRIVE: now also D1.C
- net HDD_LED_IN-: now also D1.A
- net HP_SENSEDR_A: now also D4.C
- net HP_SENSEDR_K: now also D4.A
- net MIC_SENSEDR_A: now also D3.C
- net MIC_SENSEDR_K: now also D3.A
- net PWR_LED_IN-: now also D2.A
- net SW_LED_DRIVE: now also D2.C
Other:
- moved on the sheet: J4, J5, J6, LED1B, LED1G, LED1R, R12, R13, R14, R15, R16, R17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
